File: module_swerve.kicad_sch (KiCad schematic)
At the start: 6 parts, among them J2 PlayingWFusion_CANDaisy_5-Link, M10 REV_NEO_Brushless_Motor, M11 REV_NEO_Brushless_Motor, U19 REV_Spark_MAX, U20 CTRE_CANCoder, U21 REV_Spark_MAX

Commit message: Corrections coquilles
Connections:
- new net: M11. (IN_C), U21. (VIN-)
- new net: M10. (IN_C), U19. (VIN-)
Changed lines of the file:
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@@
 		(instances
 			(project "schema_cablage_2024"
+				(path "/e63e39d7-6ac0-4ffd-8aa3-1841a4541b55/3439eb03-35bd-48b7-a9f1-5d73cc12bdd7"
+					(reference "U26")
+					(unit 1)
+				)
 				(path "/e63e39d7-6ac0-4ffd-8aa3-1841a4541b55/b632b64e-d5b7-456d-a7ae-6969aba14a97"
 					(reference "U20")
 					(unit 1)
 				)
+				(path "/e63e39d7-6ac0-4ffd-8aa3-1841a4541b55/e4b49782-05fc-4e80-9ba9-edd7f0cdce32"
+					(reference "U23")
+					(unit 1)
+				)
 				(path "/e63e39d7-6ac0-4ffd-8aa3-1841a4541b55/e92e2da7-8df4-42ea-b0b1-e2a2f3556d07"
 					(reference "U29")
-					(unit 1)
-				)
-				(path "/e63e39d7-6ac0-4ffd-8aa3-1841a4541b55/e4b49782-05fc-4e80-9ba9-edd7f0cdce32"
-					(reference "U23")
-					(unit 1)
-				)
-				(path "/e63e39d7-6ac0-4ffd-8aa3-1841a4541b55/3439eb03-35bd-48b7-a9f1-5d73cc12bdd7"
-					(reference "U26")
 					(unit 1)
 				)
@@
 		(instances
 			(project "schema_cablage_2024"
+				(path "/e63e39d7-6ac0-4ffd-8aa3-1841a4541b55/3439eb03-35bd-48b7-a9f1-5d73cc12bdd7"
+					(reference "M15")
+					(unit 1)
+				)
 				(path "/e63e39d7-6ac0-4ffd-8aa3-1841a4541b55/b632b64e-d5b7-456d-a7ae-6969aba14a97"
 					(reference "M11")
 					(unit 1)
 				)
+				(path "/e63e39d7-6ac0-4ffd-8aa3-1841a4541b55/e4b49782-05fc-4e80-9ba9-edd7f0cdce32"
+					(reference "M13")
+					(unit 1)
+				)
 				(path "/e63e39d7-6ac0-4ffd-8aa3-1841a4541b55/e92e2da7-8df4-42ea-b0b1-e2a2f3556d07"
 					(reference "M17")
-					(unit 1)
-				)
-				(path "/e63e39d7-6ac0-4ffd-8aa3-1841a4541b55/e4b49782-05fc-4e80-9ba9-edd7f0cdce32"
-					(reference "M13")
-					(unit 1)
-				)
-				(path "/e63e39d7-6ac0-4ffd-8aa3-1841a4541b55/3439eb03-35bd-48b7-a9f1-5d73cc12bdd7"
-					(reference "M15")
 					(unit 1)
 				)
@@
 		(instances
 			(project "schema_cablage_2024"
+				(path "/e63e39d7-6ac0-4ffd-8aa3-1841a4541b55/3439eb03-35bd-48b7-a9f1-5d73cc12bdd7"
+					(reference "U25")
+					(unit 1)
+				)
 				(path "/e63e39d7-6ac0-4ffd-8aa3-1841a4541b55/b632b64e-d5b7-456d-a7ae-6969aba14a97"
 					(reference "U19")
@@
 				(path "/e63e39d7-6ac0-4ffd-8aa3-1841a4541b55/e4b49782-05fc-4e80-9ba9-edd7f0cdce32"
 					(reference "U22")
-					(unit 1)
-				)
-				(path "/e63e39d7-6ac0-4ffd-8aa3-1841a4541b55/3439eb03-35bd-48b7-a9f1-5d73cc12bdd7"
-					(reference "U25")
 					(unit 1)
 				)
@@
 	)
 	(symbol
-		(lib_name "FRC_Components:REV_Spark_MAX")
 		(lib_id "FRC_Components:REV_Spark_MAX")
 		(at 96.52 107.95 270)
@@
 		(instances
 			(project "schema_cablage_2024"
+				(path "/e63e39d7-6ac0-4ffd-8aa3-1841a4541b55/3439eb03-35bd-48b7-a9f1-5d73cc12bdd7"
+					(reference "U27")
+					(unit 1)
+				)
 				(path "/e63e39d7-6ac0-4ffd-8aa3-1841a4541b55/b632b64e-d5b7-456d-a7ae-6969aba14a97"
 					(reference "U21")
@@
 				(path "/e63e39d7-6ac0-4ffd-8aa3-1841a4541b55/e4b49782-05fc-4e80-9ba9-edd7f0cdce32"
 					(reference "U24")
-					(unit 1)
-				)
-				(path "/e63e39d7-6ac0-4ffd-8aa3-1841a4541b55/3439eb03-35bd-48b7-a9f1-5d73cc12bdd7"
-					(reference "U27")
 					(unit 1)
 				)
@@
 		(instances
 			(project "schema_cablage_2024"
+				(path "/e63e39d7-6ac0-4ffd-8aa3-1841a4541b55/3439eb03-35bd-48b7-a9f1-5d73cc12bdd7"
+					(reference "J3")
+					(unit 1)
+				)
+				(path "/e63e39d7-6ac0-4ffd-8aa3-1841a4541b55/b632b64e-d5b7-456d-a7ae-6969aba14a97"
+					(reference "J1")
+					(unit 1)
+				)
 				(path "/e63e39d7-6ac0-4ffd-8aa3-1841a4541b55/e4b49782-05fc-4e80-9ba9-edd7f0cdce32"
 					(reference "J2")
-					(unit 1)
-				)
-				(path "/e63e39d7-6ac0-4ffd-8aa3-1841a4541b55/b632b64e-d5b7-456d-a7ae-6969aba14a97"
-					(reference "J1")
-					(unit 1)
-				)
-				(path "/e63e39d7-6ac0-4ffd-8aa3-1841a4541b55/3439eb03-35bd-48b7-a9f1-5d73cc12bdd7"
-					(reference "J3")
 					(unit 1)
 				)
@@
 	)
 	(symbol
-		(lib_name "FRC_Components:REV_NEO_Brushless_Motor")
 		(lib_id "FRC_Components:REV_NEO_Brushless_Motor")
 		(at 69.85 52.07 270)
@@
 		(instances
 			(project "schema_cablage_2024"
+				(path "/e63e39d7-6ac0-4ffd-8aa3-1841a4541b55/3439eb03-35bd-48b7-a9f1-5d73cc12bdd7"
+					(reference "M14")
+					(unit 1)
+				)
 				(path "/e63e39d7-6ac0-4ffd-8aa3-1841a4541b55/b632b64e-d5b7-456d-a7ae-6969aba14a97"
 					(reference "M10")
 					(unit 1)
 				)
+				(path "/e63e39d7-6ac0-4ffd-8aa3-1841a4541b55/e4b49782-05fc-4e80-9ba9-edd7f0cdce32"
+					(reference "M12")
+					(unit 1)
+				)
 				(path "/e63e39d7-6ac0-4ffd-8aa3-1841a4541b55/e92e2da7-8df4-42ea-b0b1-e2a2f3556d07"
 					(reference "M16")
 					(unit 1)
 				)
-				(path "/e63e39d7-6ac0-4ffd-8aa3-1841a4541b55/e4b49782-05fc-4e80-9ba9-edd7f0cdce32"
-					(reference "M12")
-					(unit 1)
-				)
-				(path "/e63e39d7-6ac0-4ffd-8aa3-1841a4541b55/3439eb03-35bd-48b7-a9f1-5d73cc12bdd7"
-					(reference "M14")
-					(unit 1)
-				)
